Commit message: wip: 6-joints wheel system

File: hamster_vehicle_description/urdf/front_wheel.urdf.xacro (robot description, xacro)
@@ -1,4 +1,4 @@
 <?xml version="1.0"?>
-<robot name="wheel" xmlns:xacro="http://www.ros.org/wiki/xacro">
+<robot name="front_wheel" xmlns:xacro="http://www.ros.org/wiki/xacro">
   <!-- Wheels -->
   <xacro:property name="wheel_radius" value="0.029" />
@@ -15,4 +15,23 @@
   <xacro:macro name="wheel" params="fr lr parent origin_x origin_y origin_z"> <!--fr : front, rear ; lr: left, right -->
     <link name="${fr}_${lr}_wheel">
+      <visual>
+        <origin xyz="0 0 0" rpy="1.57 0 0" />
+        <geometry>
+          <box size="0.01 0.01 0.01" />
+        </geometry>
+      </visual>
+      <collision>
+        <origin xyz="0 0 0" rpy="1.57 0 0" />
+        <geometry>
+          <cylinder length="${wheel_height}" radius="${wheel_radius}" />
+        </geometry>
+      </collision>
+      <inertial>
+        <mass value="${wheel_mass}" />
+        <origin xyz="0 0 0" rpy="1.57 0 0" />
+        <cylinder_inertia  m="${wheel_mass}" r="${wheel_radius}" h="${wheel_height}" />
+      </inertial>
+    </link>
+    <link name="${fr}_${lr}_wheel_steering">
       <visual>
         <origin xyz="0 0 0" rpy="1.57 0 0" />
@@ -54,4 +73,11 @@
       <!-- <dynamics damping="0.7"/> -->
     </joint>
+        <joint name="${fr}_${lr}_wheel_steering_joint" type="continuous">
+      <parent link="${parent}"/>
+      <child link="${fr}_${lr}_wheel_steering"/>
+      <origin xyz="${origin_x} ${origin_y} ${origin_z}" rpy="0 0 0" />
+      <axis xyz="0 0 1" rpy="0 0 0" />
+      <!-- <dynamics damping="0.7"/> -->
+    </joint>
     <!-- Transmission is important to link the joints and the controller -->
     <transmission name="${fr}_${lr}_wheel_joint_trans">

File: hamster_vehicle_description/urdf/hamster.urdf.xacro (robot description, xacro)
@@ -1,5 +1,6 @@
 <?xml version="1.0"?>
 <robot name="hamster" xmlns:xacro="http://www.ros.org/wiki/xacro">
-  <xacro:include filename="$(find hamster_vehicle_description)/urdf/wheel.urdf.xacro" />
+  <xacro:include filename="$(find hamster_vehicle_description)/urdf/front_wheel.urdf.xacro" />
+  <xacro:include filename="$(find hamster_vehicle_description)/urdf/rear_wheel.urdf.xacro" />
   <xacro:macro name="solid_cuboid_inertia" params="w h d m">
   <inertia  ixx="${m*(h*h+d*d)/12}" ixy = "0" ixz = "0"
@@ -28,8 +29,9 @@
     <collision>
       <geometry>
-        <box size="0.25 0.09 0.05" />
+        <box size="0.25 0.09 0.02" />
       </geometry>
     </collision>
   </link>
+<!--
   <link name="imu_link">
     <inertial>
@@ -42,5 +44,6 @@
       </geometry>
     </visual>
-    </link>
+    </link> -->
+<!--
   <joint name="imu_link_joint" type="fixed">
     <origin xyz="0 0 0" rpy="0 0 0" />
@@ -59,7 +62,7 @@
     <parent link="base_link"/>
     <child link="camera_link"/>
-  </joint>
+  </joint> -->
   <!-- Hokuyo Laser -->
-  <link name="lidar_link">
+  <!-- <link name="lidar_link">
     <collision>
       <geometry>
@@ -76,6 +79,6 @@
       <inertia ixx="1e-6" ixy="0" ixz="0" iyy="1e-6" iyz="0" izz="1e-6" />
     </inertial>
-  </link>
-    <link name="camera_link">
+  </link> -->
+  <!-- <link name="camera_link">
     <collision>
       <geometry>
@@ -93,19 +96,9 @@
       <inertia ixx="1e-6" ixy="0" ixz="0" iyy="1e-6" iyz="0" izz="1e-6" />
     </inertial>
-  </link>
-  <wheel fr="front" lr="right" parent="base_link" origin_x="0.08" origin_y="-0.086" origin_z="-0.01"/>
-  <wheel fr="front" lr="left" parent="base_link" origin_x="0.08" origin_y="0.086" origin_z="-0.01"/>
-  <wheel fr="rear" lr="right" parent="base_link" origin_x="-0.085" origin_y="-0.086" origin_z="-0.01"/>
-  <wheel fr="rear" lr="left" parent="base_link" origin_x="-0.085" origin_y="0.086" origin_z="-0.01"/>
-  <joint name="front_right_wheel_steering_joint" type="continuous">
-    <parent link="${parent}"/>
-    <child link="front_right_wheel_steering"/>
-    <axis xyz="0 0 0" rpy="0 0 0" />
-  </joint>
-  <joint name="front_left_wheel_steering_joint" type="continuous">
-    <parent link="${parent}"/>
-    <child link="front_left_wheel_steering"/>
-    <axis xyz="0 0 0" rpy="0 0 0" />
-  </joint>
+  </link> -->
+  <front_wheel fr="front" lr="right" parent="base_link" origin_x="0.08" origin_y="-0.086" origin_z="-0.01"/>
+  <front_wheel fr="front" lr="left" parent="base_link" origin_x="0.08" origin_y="0.086" origin_z="-0.01"/>
+  <!-- <rear_wheel fr="rear" lr="right" parent="base_link" origin_x="-0.085" origin_y="-0.086" origin_z="-0.01"/> -->
+  <!-- <rear_wheel fr="rear" lr="left" parent="base_link" origin_x="-0.085" origin_y="0.086" origin_z="-0.01"/>  -->
   <gazebo>
     <plugin name="gazebo_ros_control" filename="libgazebo_ros_control.so">
@@ -116,28 +109,10 @@
   </gazebo>
             <!-- Skid steer drive controller -->
-  <gazebo>
-    <!-- <plugin name="skid_steer_drive_controller" filename="libgazebo_ros_skid_steer_drive.so">
-      <alwaysOn>1</alwaysOn>
-      <updateRate>100.0</updateRate>
+  <!-- <gazebo>
+    <plugin name="gazebo_ackermann_drive" filename="libgazebo_ackermann_drive.so" >
       <robotNamespace>$(arg agent)</robotNamespace>
-      <leftFrontJoint>front_left_wheel_joint</leftFrontJoint>
-      <rightFrontJoint>front_right_wheel_joint</rightFrontJoint>
-      <leftRearJoint>rear_left_wheel_joint</leftRearJoint>
-      <rightRearJoint>rear_right_wheel_joint</rightRearJoint>
-      <wheelSeparation>0.18</wheelSeparation>
-      <wheelDiameter>0.058</wheelDiameter>
-      <torque>50</torque>
-      <broadcastTF>0</broadcastTF>
-      <odometryFrame>map</odometryFrame>
-      <commandTopic>cmd_vel</commandTopic>
-      <odometryTopic>odom</odometryTopic>
-      <robotBaseFrame>base_link</robotBaseFrame>
-      <covariance_x>0.0001</covariance_x>
-      <covariance_y>0.0001</covariance_y>
-      <covariance_z>0.0001</covariance_z>
-      <covariance_yaw>0.0001</covariance_yaw>
-    </plugin> -->
-  </gazebo>
-  <gazebo reference="imu_link">
+    </plugin>
+  </gazebo> -->
+  <!-- <gazebo reference="imu_link">
     <gravity>true</gravity>
     <sensor name="imu_sensor" type="imu">
@@ -156,6 +131,6 @@
       </plugin>
     </sensor>
-  </gazebo>
-  <gazebo reference="lidar_link">
+  </gazebo> -->
+  <!-- <gazebo reference="lidar_link">
     <sensor type="gpu_ray" name="head_hokuyo_sensor">
       <pose>0 0 0 0 0 0</pose>
@@ -187,6 +162,6 @@
       </plugin>
     </sensor>
-  </gazebo>
-  <gazebo reference="camera_link">
+  </gazebo> -->
+  <!-- <gazebo reference="camera_link">
     <sensor name="depth_camera" type="depth">
       <update_rate>15</update_rate>
@@ -228,4 +203,4 @@
       </plugin>
     </sensor>
-  </gazebo>
+  </gazebo> -->
 </robot>

Commit message: wip:joints pid

File: hamster_vehicle_description/urdf/front_wheel.urdf.xacro (robot description, xacro)
@@ -13,10 +13,10 @@
               izz="${m*r*r/2}" />
   </xacro:macro>
-  <xacro:macro name="wheel" params="fr lr parent origin_x origin_y origin_z"> <!--fr : front, rear ; lr: left, right -->
+  <xacro:macro name="front_wheel" params="fr lr parent origin_x origin_y origin_z"> <!--fr : front, rear ; lr: left, right -->
     <link name="${fr}_${lr}_wheel">
       <visual>
         <origin xyz="0 0 0" rpy="1.57 0 0" />
         <geometry>
-          <box size="0.01 0.01 0.01" />
+          <mesh filename="package://hamster_vehicle_description/meshes/wheel.dae" />
         </geometry>
       </visual>
@@ -34,15 +34,14 @@
     </link>
     <link name="${fr}_${lr}_wheel_steering">
-      <visual>
+      <!-- <visual>
         <origin xyz="0 0 0" rpy="1.57 0 0" />
         <geometry>
-          <!-- <cylinder length="${wheel_height}" radius="${wheel_radius}" /> -->
           <mesh filename="package://hamster_vehicle_description/meshes/wheel.dae" />
         </geometry>
-      </visual>
+      </visual> -->
       <collision>
-        <origin xyz="0 0 0" rpy="1.57 0 0" />
+        <origin xyz="0 0.02 0" rpy="1.57 0 0" />
         <geometry>
-          <cylinder length="${wheel_height}" radius="${wheel_radius}" />
+          <cylinder length="0.001" radius="0.001" />
         </geometry>
       </collision>
@@ -67,11 +66,11 @@
     </gazebo>
     <joint name="${fr}_${lr}_wheel_joint" type="continuous">
-      <parent link="${parent}"/>
+      <parent link="${fr}_${lr}_wheel_steering"/>
       <child link="${fr}_${lr}_wheel"/>
-      <origin xyz="${origin_x} ${origin_y} ${origin_z}" rpy="0 0 0" />
+      <origin xyz="0 0 0" rpy="0 0 0" />
       <axis xyz="0 1 0" rpy="0 0 0" />
       <!-- <dynamics damping="0.7"/> -->
     </joint>
-        <joint name="${fr}_${lr}_wheel_steering_joint" type="continuous">
+    <joint name="${fr}_${lr}_wheel_steering_joint" type="continuous">
       <parent link="${parent}"/>
       <child link="${fr}_${lr}_wheel_steering"/>

File: hamster_vehicle_description/urdf/hamster.urdf.xacro (robot description, xacro)
@@ -9,4 +9,5 @@
   </xacro:macro>
   <xacro:arg name="agent" default="agent1" />
+  <link name="dummy"/>
   <link name="base_link">
     <inertial>
@@ -33,5 +34,4 @@
     </collision>
   </link>
-<!--
   <link name="imu_link">
     <inertial>
@@ -44,6 +44,10 @@
       </geometry>
     </visual>
-    </link> -->
-<!--
+    </link>
+  <joint name="dummy_link_joint" type="fixed">
+    <origin xyz="0 0 0" rpy="0 0 0" />
+    <parent link="dummy" />
+    <child  link="base_link" />
+  </joint>
   <joint name="imu_link_joint" type="fixed">
     <origin xyz="0 0 0" rpy="0 0 0" />
@@ -62,7 +66,7 @@
     <parent link="base_link"/>
     <child link="camera_link"/>
-  </joint> -->
+  </joint>
   <!-- Hokuyo Laser -->
-  <!-- <link name="lidar_link">
+  <link name="lidar_link">
     <collision>
       <geometry>
@@ -79,6 +83,6 @@
       <inertia ixx="1e-6" ixy="0" ixz="0" iyy="1e-6" iyz="0" izz="1e-6" />
     </inertial>
-  </link> -->
-  <!-- <link name="camera_link">
+  </link>
+  <link name="camera_link">
     <collision>
       <geometry>
@@ -96,9 +100,9 @@
       <inertia ixx="1e-6" ixy="0" ixz="0" iyy="1e-6" iyz="0" izz="1e-6" />
     </inertial>
-  </link> -->
+  </link>
   <front_wheel fr="front" lr="right" parent="base_link" origin_x="0.08" origin_y="-0.086" origin_z="-0.01"/>
   <front_wheel fr="front" lr="left" parent="base_link" origin_x="0.08" origin_y="0.086" origin_z="-0.01"/>
-  <!-- <rear_wheel fr="rear" lr="right" parent="base_link" origin_x="-0.085" origin_y="-0.086" origin_z="-0.01"/> -->
-  <!-- <rear_wheel fr="rear" lr="left" parent="base_link" origin_x="-0.085" origin_y="0.086" origin_z="-0.01"/>  -->
+  <rear_wheel fr="rear" lr="right" parent="base_link" origin_x="-0.085" origin_y="-0.086" origin_z="-0.01"/>
+  <rear_wheel fr="rear" lr="left" parent="base_link" origin_x="-0.085" origin_y="0.086" origin_z="-0.01"/>
   <gazebo>
     <plugin name="gazebo_ros_control" filename="libgazebo_ros_control.so">
@@ -109,10 +113,10 @@
   </gazebo>
             <!-- Skid steer drive controller -->
-  <!-- <gazebo>
+  <gazebo>
     <plugin name="gazebo_ackermann_drive" filename="libgazebo_ackermann_drive.so" >
       <robotNamespace>$(arg agent)</robotNamespace>
     </plugin>
-  </gazebo> -->
-  <!-- <gazebo reference="imu_link">
+  </gazebo>
+  <gazebo reference="imu_link">
     <gravity>true</gravity>
     <sensor name="imu_sensor" type="imu">
@@ -131,6 +135,6 @@
       </plugin>
     </sensor>
-  </gazebo> -->
-  <!-- <gazebo reference="lidar_link">
+  </gazebo>
+  <gazebo reference="lidar_link">
     <sensor type="gpu_ray" name="head_hokuyo_sensor">
       <pose>0 0 0 0 0 0</pose>
@@ -162,6 +166,6 @@
       </plugin>
     </sensor>
-  </gazebo> -->
-  <!-- <gazebo reference="camera_link">
+  </gazebo>
+  <gazebo reference="camera_link">
     <sensor name="depth_camera" type="depth">
       <update_rate>15</update_rate>
@@ -203,4 +207,4 @@
       </plugin>
     </sensor>
-  </gazebo> -->
+  </gazebo>
 </robot>

File: hamster_vehicle_description/urdf/rear_wheel.urdf.xacro (robot description, xacro)
@@ -13,5 +13,5 @@
               izz="${m*r*r/2}" />
   </xacro:macro>
-  <xacro:macro name="wheel" params="fr lr parent origin_x origin_y origin_z"> <!--fr : front, rear ; lr: left, right -->
+  <xacro:macro name="rear_wheel" params="fr lr parent origin_x origin_y origin_z"> <!--fr : front, rear ; lr: left, right -->
     <link name="${fr}_${lr}_wheel">
       <visual>
@@ -51,4 +51,6 @@
       <origin xyz="${origin_x} ${origin_y} ${origin_z}" rpy="0 0 0" />
       <axis xyz="0 1 0" rpy="0 0 0" />
+      <limit effort="30" velocity="1.2"/>
+      <dynamics friction="0.0"/>
       <!-- <dynamics damping="0.7"/> -->
     </joint>

Commit message: wip:velocity calc todo

File: hamster_vehicle_description/urdf/front_wheel.urdf.xacro (robot description, xacro)
@@ -41,5 +41,5 @@
       </visual> -->
       <collision>
-        <origin xyz="0 0.02 0" rpy="1.57 0 0" />
+        <origin xyz="0 0.02 0" rpy="0 0 0" />
         <geometry>
           <cylinder length="0.001" radius="0.001" />
@@ -47,7 +47,7 @@
       </collision>
       <inertial>
-        <mass value="${wheel_mass}" />
-        <origin xyz="0 0 0" rpy="1.57 0 0" />
-        <cylinder_inertia  m="${wheel_mass}" r="${wheel_radius}" h="${wheel_height}" />
+        <mass value="0.1" />
+        <origin xyz="0 0 0" rpy="0 0 0" />
+        <cylinder_inertia  m="0.1" r="0.01" h="0.01" />
       </inertial>
     </link>
@@ -70,5 +70,6 @@
       <origin xyz="0 0 0" rpy="0 0 0" />
       <axis xyz="0 1 0" rpy="0 0 0" />
-      <!-- <dynamics damping="0.7"/> -->
+      <limit effort="1" velocity="1.5"/>
+      <!-- <dynamics friction="0.5" damping="0.7" /> -->
     </joint>
     <joint name="${fr}_${lr}_wheel_steering_joint" type="continuous">
@@ -77,8 +78,9 @@
       <origin xyz="${origin_x} ${origin_y} ${origin_z}" rpy="0 0 0" />
       <axis xyz="0 0 1" rpy="0 0 0" />
+      <limit effort="1" velocity="1.5"/>
       <!-- <dynamics damping="0.7"/> -->
     </joint>
     <!-- Transmission is important to link the joints and the controller -->
-    <transmission name="${fr}_${lr}_wheel_joint_trans">
+    <!-- <transmission name="${fr}_${lr}_wheel_joint_trans">
       <type>transmission_interface/SimpleTransmission</type>
       <joint name="${fr}_${lr}_wheel_joint">
@@ -89,5 +91,5 @@
         <mechanicalReduction>1</mechanicalReduction>
       </actuator>
-    </transmission>
+    </transmission> -->
   </xacro:macro>
 </robot>

File: hamster_vehicle_description/urdf/hamster.urdf.xacro (robot description, xacro)
@@ -13,5 +13,5 @@
     <inertial>
       <mass value="1.0" />
-      <solid_cuboid_inertia w="0.1" h="0.1" d="0.2" m="1.0"/>
+      <solid_cuboid_inertia w="0.1" h="0.1" d="0.1" m="1.0"/>
     </inertial>
     <surface>

File: hamster_vehicle_description/urdf/rear_wheel.urdf.xacro (robot description, xacro)
@@ -51,10 +51,9 @@
       <origin xyz="${origin_x} ${origin_y} ${origin_z}" rpy="0 0 0" />
       <axis xyz="0 1 0" rpy="0 0 0" />
-      <limit effort="30" velocity="1.2"/>
-      <dynamics friction="0.0"/>
-      <!-- <dynamics damping="0.7"/> -->
+      <limit effort="1" velocity="1.5"/>
+      <!-- <dynamics friction="0.5" damping="0.7" /> -->
     </joint>
     <!-- Transmission is important to link the joints and the controller -->
-    <transmission name="${fr}_${lr}_wheel_joint_trans">
+    <!-- <transmission name="${fr}_${lr}_wheel_joint_trans">
       <type>transmission_interface/SimpleTransmission</type>
       <joint name="${fr}_${lr}_wheel_joint">
@@ -65,5 +64,5 @@
         <mechanicalReduction>1</mechanicalReduction>
       </actuator>
-    </transmission>
+    </transmission> -->
   </xacro:macro>
 </robot>
