Commit message: speed and friction fixed, V6/7 added, worlds added

File: hamster_vehicle_description/urdf/front_wheel.urdf.xacro (robot description, xacro)
@@ -5,7 +5,4 @@
   <xacro:property name="wheel_height" value="0.02" />
   <xacro:property name="wheel_mass" value="0.1" /> <!-- in kg-->
-  <!-- <xacro:property name="base_x_origin_to_wheel_origin" value="0.25" />
-  <xacro:property name="base_y_origin_to_wheel_origin" value="0.3" />
-  <xacro:property name="base_z_origin_to_wheel_origin" value="0.0" /> -->
   <xacro:macro name="cylinder_inertia" params="m r h">
     <inertia  ixx="${m*(3*r*r+h*h)/12}" ixy="0" ixz="0"
@@ -34,10 +31,4 @@
     </link>
     <link name="${fr}_${lr}_wheel_steering">
-      <!-- <visual>
-        <origin xyz="0 0 0" rpy="1.57 0 0" />
-        <geometry>
-          <mesh filename="package://hamster_vehicle_description/meshes/wheel.dae" />
-        </geometry>
-      </visual> -->
       <collision>
         <origin xyz="0 0.02 0" rpy="0 0 0" />
@@ -53,15 +44,10 @@
     </link>
     <gazebo reference="${fr}_${lr}_wheel">
-     <collision>
-      <surface>
-        <friction>
-          <torsional>
-            <coefficient>0.1</coefficient>
-            <use_patch_radius>false</use_patch_radius>
-            <patch_radius>0.05</patch_radius>
-          </torsional>
-        </friction>
-      </surface>
-     </collision>
+      <mu1>70</mu1>
+      <mu2>70</mu2>
+      <dampingFactor>0.1</dampingFactor>
+      <minDepth>0.01</minDepth>
+      <selfCollide>false</selfCollide>
+      <maxContacts>20</maxContacts>
     </gazebo>
     <joint name="${fr}_${lr}_wheel_joint" type="continuous">
@@ -78,18 +64,7 @@
       <origin xyz="${origin_x} ${origin_y} ${origin_z}" rpy="0 0 0" />
       <axis xyz="0 0 1" rpy="0 0 0" />
-      <limit effort="1" velocity="1.5"/>
+      <limit effort="30" velocity="1.5" lower="-0.296706" upper="0.296706"/>
       <!-- <dynamics damping="0.7"/> -->
     </joint>
-    <!-- Transmission is important to link the joints and the controller -->
-    <!-- <transmission name="${fr}_${lr}_wheel_joint_trans">
-      <type>transmission_interface/SimpleTransmission</type>
-      <joint name="${fr}_${lr}_wheel_joint">
-          <hardwareInterface>hardware_interface/EffortJointInterface</hardwareInterface>
-      </joint>
-      <actuator name="${fr}_${lr}_wheel_joint_motor">
-        <hardwareInterface>hardware_interface/EffortJointInterface</hardwareInterface>
-        <mechanicalReduction>1</mechanicalReduction>
-      </actuator>
-    </transmission> -->
   </xacro:macro>
 </robot>

File: hamster_vehicle_description/urdf/hamster.urdf.xacro (robot description, xacro)
@@ -9,4 +9,6 @@
   </xacro:macro>
   <xacro:arg name="agent" default="agent1" />
+  <xacro:arg name="robot_version" default="V6"/>
+  <xacro:property name="version" value="$(arg robot_version)"/>
   <link name="dummy"/>
   <link name="base_link">
@@ -15,12 +17,4 @@
       <solid_cuboid_inertia w="0.1" h="0.1" d="0.1" m="1.0"/>
     </inertial>
-    <surface>
-      <friction>
-        <ode>
-          <mu>1.0</mu>
-          <mu2>1.0</mu2>
-        </ode>
-      </friction>
-    </surface>
     <visual>
       <geometry>
@@ -63,5 +57,10 @@
   <joint name="camera_joint" type="fixed">
     <axis xyz="0 1 0" />
-    <origin xyz="0.12673 0 0.028" rpy="1.57 0 1.57"/>
+    <xacro:if value="${version == 'V7'}">
+      <origin xyz="0.12673 0 0.028" rpy="1.57 0 1.57"/>
+    </xacro:if>
+      <xacro:if value="${version == 'V6'}">
+      <origin xyz="0.1 0 0.02" rpy="0 0 0"/>
+    </xacro:if>
     <parent link="base_link"/>
     <child link="camera_link"/>
@@ -92,5 +91,10 @@
     <visual>
       <geometry>
+        <xacro:if value="${version == 'V7'}">
         <mesh filename="package://hamster_vehicle_description/meshes/d415.stl" />
+        </xacro:if>
+        <xacro:if value="${version == 'V6'}">
+        <mesh filename="package://hamster_vehicle_description/meshes/camera.stl" />
+        </xacro:if>
       </geometry>
       <material name="red"/>
@@ -167,44 +171,87 @@
     </sensor>
   </gazebo>
-  <gazebo reference="camera_link">
-    <sensor name="depth_camera" type="depth">
-      <update_rate>15</update_rate>
-      <camera>
-        <horizontal_fov>1.5882496</horizontal_fov>
-        <image>
-          <width>640</width>
-          <height>480</height>
-          <format>R8G8B8</format>
-        </image>
-        <clip>
-          <near>0.05</near>
-          <far>3</far>
-        </clip>
-      </camera>
-      <plugin name="camera_controller" filename="libgazebo_ros_openni_kinect.so">
-        <baseline>0.2</baseline>
-        <alwaysOn>true</alwaysOn>
-        <updateRate>1.0</updateRate>
-        <cameraName>$(arg agent)</cameraName>
-        <imageTopicName>camera/color/image_raw</imageTopicName>
-        <cameraInfoTopicName>camera/color/camera_info</cameraInfoTopicName>
-        <depthImageTopicName>camera/depth/image_raw</depthImageTopicName>
-        <depthImageInfoTopicName>camera/depth/camera_info</depthImageInfoTopicName>
-        <pointCloudTopicName>camera/depth/points</pointCloudTopicName>
-        <frameName>$(arg agent)/camera_link</frameName>
-        <pointCloudCutoff>0.5</pointCloudCutoff>
-        <pointCloudCutoffMax>3.0</pointCloudCutoffMax>
-        <distortionK1>0.00000001</distortionK1>
-        <distortionK2>0.00000001</distortionK2>
-        <distortionK3>0.00000001</distortionK3>
-        <distortionT1>0.00000001</distortionT1>
-        <distortionT2>0.00000001</distortionT2>
-        <CxPrime>0</CxPrime>
-        <Cx>0</Cx>
-        <Cy>0</Cy>
-        <focalLength>0</focalLength>
-        <hackBaseline>0</hackBaseline>
-      </plugin>
-    </sensor>
-  </gazebo>
+  <xacro:if value="${version == 'V7'}">
+    <gazebo reference="camera_link">
+      <sensor name="depth_camera" type="depth">
+        <update_rate>15</update_rate>
+        <camera>
+          <horizontal_fov>1.5882496</horizontal_fov>
+          <image>
+            <width>640</width>
+            <height>480</height>
+            <format>R8G8B8</format>
+          </image>
+          <clip>
+            <near>0.05</near>
+            <far>3</far>
+          </clip>
+        </camera>
+        <plugin name="camera_controller" filename="libgazebo_ros_openni_kinect.so">
+          <baseline>0.2</baseline>
+          <alwaysOn>true</alwaysOn>
+          <updateRate>1.0</updateRate>
+          <cameraName>$(arg agent)</cameraName>
+          <imageTopicName>camera/color/image_raw</imageTopicName>
+          <cameraInfoTopicName>camera/color/camera_info</cameraInfoTopicName>
+          <depthImageTopicName>camera/depth/image_raw</depthImageTopicName>
+          <depthImageInfoTopicName>camera/depth/camera_info</depthImageInfoTopicName>
+          <pointCloudTopicName>camera/depth/points</pointCloudTopicName>
+          <frameName>$(arg agent)/camera_link</frameName>
+          <pointCloudCutoff>0.5</pointCloudCutoff>
+          <pointCloudCutoffMax>3.0</pointCloudCutoffMax>
+          <distortionK1>0.00000001</distortionK1>
+          <distortionK2>0.00000001</distortionK2>
+          <distortionK3>0.00000001</distortionK3>
+          <distortionT1>0.00000001</distortionT1>
+          <distortionT2>0.00000001</distortionT2>
+          <CxPrime>0</CxPrime>
+          <Cx>0</Cx>
+          <Cy>0</Cy>
+          <focalLength>0</focalLength>
+          <hackBaseline>0</hackBaseline>
+        </plugin>
+      </sensor>
+    </gazebo>
+  </xacro:if>
+  <xacro:if value="${version == 'V6'}">
+    <gazebo reference="camera_link">
+      <sensor type="camera" name="camera1">
+        <update_rate>30.0</update_rate>
+        <camera name="head">
+          <horizontal_fov>1.3962634</horizontal_fov>
+          <image>
+            <width>800</width>
+            <height>800</height>
+            <format>R8G8B8</format>
+          </image>
+          <clip>
+            <near>0.02</near>
+            <far>300</far>
+          </clip>
+          <noise>
+            <type>gaussian</type>
+            <!-- Noise is sampled independently per pixel on each frame.
+                 That pixel's noise value is added to each of its color
+                 channels, which at that point lie in the range [0,1]. -->
+            <mean>0.0</mean>
+            <stddev>0.007</stddev>
+          </noise>
+        </camera>
+        <plugin name="camera_controller" filename="libgazebo_ros_camera.so">
+          <alwaysOn>true</alwaysOn>
+          <updateRate>0.0</updateRate>
+          <cameraName>$(arg agent)</cameraName>
+          <imageTopicName>image_raw</imageTopicName>
+          <cameraInfoTopicName>camera_info</cameraInfoTopicName>
+          <frameName>$(arg agent)/camera_link</frameName>
+          <hackBaseline>0.07</hackBaseline>
+          <distortionK1>0.0</distortionK1>
+          <distortionK2>0.0</distortionK2>
+          <distortionK3>0.0</distortionK3>
+          <distortionT1>0.0</distortionT1>
+          <distortionT2>0.0</distortionT2>
+        </plugin>
+      </sensor>
+    </gazebo>
+  </xacro:if>
 </robot>

File: hamster_vehicle_description/urdf/rear_wheel.urdf.xacro (robot description, xacro)
@@ -5,7 +5,4 @@
   <xacro:property name="wheel_height" value="0.02" />
   <xacro:property name="wheel_mass" value="0.1" /> <!-- in kg-->
-  <!-- <xacro:property name="base_x_origin_to_wheel_origin" value="0.25" />
-  <xacro:property name="base_y_origin_to_wheel_origin" value="0.3" />
-  <xacro:property name="base_z_origin_to_wheel_origin" value="0.0" /> -->
   <xacro:macro name="cylinder_inertia" params="m r h">
     <inertia  ixx="${m*(3*r*r+h*h)/12}" ixy="0" ixz="0"
@@ -34,15 +31,10 @@
     </link>
     <gazebo reference="${fr}_${lr}_wheel">
-     <collision>
-      <surface>
-        <friction>
-          <torsional>
-            <coefficient>0.1</coefficient>
-            <use_patch_radius>false</use_patch_radius>
-            <patch_radius>0.05</patch_radius>
-          </torsional>
-        </friction>
-      </surface>
-     </collision>
+      <mu1>70</mu1>
+      <mu2>70</mu2>
+      <dampingFactor>0.1</dampingFactor>
+      <minDepth>0.01</minDepth>
+      <selfCollide>false</selfCollide>
+      <maxContacts>20</maxContacts>
     </gazebo>
     <joint name="${fr}_${lr}_wheel_joint" type="continuous">
@@ -51,18 +43,7 @@
       <origin xyz="${origin_x} ${origin_y} ${origin_z}" rpy="0 0 0" />
       <axis xyz="0 1 0" rpy="0 0 0" />
-      <limit effort="1" velocity="1.5"/>
+      <limit effort="30" velocity="1.5"/>
       <!-- <dynamics friction="0.5" damping="0.7" /> -->
     </joint>
-    <!-- Transmission is important to link the joints and the controller -->
-    <!-- <transmission name="${fr}_${lr}_wheel_joint_trans">
-      <type>transmission_interface/SimpleTransmission</type>
-      <joint name="${fr}_${lr}_wheel_joint">
-          <hardwareInterface>hardware_interface/EffortJointInterface</hardwareInterface>
-      </joint>
-      <actuator name="${fr}_${lr}_wheel_joint_motor">
-        <hardwareInterface>hardware_interface/EffortJointInterface</hardwareInterface>
-        <mechanicalReduction>1</mechanicalReduction>
-      </actuator>
-    </transmission> -->
   </xacro:macro>
 </robot>

Commit message: odometry tf added, wheels improved

File: hamster_vehicle_description/urdf/front_wheel.urdf.xacro (robot description, xacro)
@@ -15,5 +15,5 @@
         <origin xyz="0 0 0" rpy="1.57 0 0" />
         <geometry>
-          <mesh filename="package://hamster_vehicle_description/meshes/wheel.dae" />
+          <mesh filename="package://hamster_vehicle_description/meshes/hamster_wheel.dae" />
         </geometry>
       </visual>
@@ -21,5 +21,5 @@
         <origin xyz="0 0 0" rpy="1.57 0 0" />
         <geometry>
-          <cylinder length="${wheel_height}" radius="${wheel_radius}" />
+          <cylinder length="0.008" radius="${wheel_radius}" />
         </geometry>
       </collision>
@@ -43,11 +43,22 @@
       </inertial>
     </link>
-    <gazebo reference="${fr}_${lr}_wheel">
-      <mu1>70</mu1>
-      <mu2>70</mu2>
+    <!-- <gazebo reference="${fr}_${lr}_wheel">
+      <mu1>100</mu1>
+      <mu2>100</mu2>
       <dampingFactor>0.1</dampingFactor>
       <minDepth>0.01</minDepth>
       <selfCollide>false</selfCollide>
       <maxContacts>20</maxContacts>
+    </gazebo> -->
+    <gazebo reference="${fr}_${lr}_wheel">
+      <mu1>0.7</mu1>
+      <mu2>0.7</mu2>
+      <kp>500000.0</kp>
+      <kd>10.0</kd>
+      <minDepth>0.002</minDepth>
+      <maxVel>0.1</maxVel>
+      <fdir1>1 0 0</fdir1>
+      <maxContacts>20</maxContacts>
+      <!-- <material>Gazebo/FlatBlack</material> -->
     </gazebo>
     <joint name="${fr}_${lr}_wheel_joint" type="continuous">
@@ -56,5 +67,5 @@
       <origin xyz="0 0 0" rpy="0 0 0" />
       <axis xyz="0 1 0" rpy="0 0 0" />
-      <limit effort="1" velocity="1.5"/>
+      <limit effort="-1" velocity="-1"/>
       <!-- <dynamics friction="0.5" damping="0.7" /> -->
     </joint>

File: hamster_vehicle_description/urdf/hamster.urdf.xacro (robot description, xacro)
@@ -11,9 +11,9 @@
   <xacro:arg name="robot_version" default="V6"/>
   <xacro:property name="version" value="$(arg robot_version)"/>
-  <link name="dummy"/>
+  <!-- <link name="dummy"/> -->
   <link name="base_link">
     <inertial>
-      <mass value="1.0" />
-      <solid_cuboid_inertia w="0.1" h="0.1" d="0.1" m="1.0"/>
+      <mass value="3.0" />
+      <solid_cuboid_inertia w="0.1" h="0.1" d="0.3" m="3.0"/>
     </inertial>
     <visual>
@@ -39,9 +39,9 @@
     </visual>
     </link>
-  <joint name="dummy_link_joint" type="fixed">
+  <!-- <joint name="dummy_link_joint" type="fixed">
     <origin xyz="0 0 0" rpy="0 0 0" />
     <parent link="dummy" />
     <child  link="base_link" />
-  </joint>
+  </joint> -->
   <joint name="imu_link_joint" type="fixed">
     <origin xyz="0 0 0" rpy="0 0 0" />
@@ -130,5 +130,5 @@
       <topic>__default_topic__</topic>
       <plugin filename="libgazebo_ros_imu_sensor.so" name="imu_plugin">
-        <topicName>$(arg agent)/imu</topicName>
+        <topicName>imu</topicName>
         <bodyName>imu_link</bodyName>
         <updateRateHZ>10.0</updateRateHZ>
@@ -148,5 +148,5 @@
         <scan>
           <horizontal>
-            <samples>720</samples>
+            <samples>360</samples>
             <resolution>1</resolution>
             <min_angle>-3.1415</min_angle>
@@ -166,5 +166,5 @@
       </ray>
       <plugin name="gazebo_ros_head_hokuyo_controller" filename="libgazebo_ros_gpu_laser.so">
-        <topicName>$(arg agent)/scan</topicName>
+        <topicName>scan</topicName>
         <frameName>$(arg agent)/lidar_link</frameName>
       </plugin>
@@ -191,5 +191,5 @@
           <alwaysOn>true</alwaysOn>
           <updateRate>1.0</updateRate>
-          <cameraName>$(arg agent)</cameraName>
+          <cameraName></cameraName>
           <imageTopicName>camera/color/image_raw</imageTopicName>
           <cameraInfoTopicName>camera/color/camera_info</cameraInfoTopicName>
@@ -241,5 +241,5 @@
           <alwaysOn>true</alwaysOn>
           <updateRate>0.0</updateRate>
-          <cameraName>$(arg agent)</cameraName>
+          <cameraName></cameraName>
           <imageTopicName>image_raw</imageTopicName>
           <cameraInfoTopicName>camera_info</cameraInfoTopicName>

File: hamster_vehicle_description/urdf/rear_wheel.urdf.xacro (robot description, xacro)
@@ -15,5 +15,5 @@
         <origin xyz="0 0 0" rpy="1.57 0 0" />
         <geometry>
-          <mesh filename="package://hamster_vehicle_description/meshes/wheel.dae" />
+          <mesh filename="package://hamster_vehicle_description/meshes/hamster_wheel.dae" />
         </geometry>
       </visual>
@@ -21,5 +21,5 @@
         <origin xyz="0 0 0" rpy="1.57 0 0" />
         <geometry>
-          <cylinder length="${wheel_height}" radius="${wheel_radius}" />
+          <cylinder length="0.008" radius="${wheel_radius}" />
         </geometry>
       </collision>
@@ -30,10 +30,21 @@
       </inertial>
     </link>
-    <gazebo reference="${fr}_${lr}_wheel">
-      <mu1>70</mu1>
-      <mu2>70</mu2>
+    <!-- <gazebo reference="${fr}_${lr}_wheel">
+      <mu1>100</mu1>
+      <mu2>100</mu2>
       <dampingFactor>0.1</dampingFactor>
       <minDepth>0.01</minDepth>
       <selfCollide>false</selfCollide>
+      <maxContacts>20</maxContacts>
+    </gazebo> -->
+    <gazebo reference="${fr}_${lr}_wheel">
+      <mu1>0.7</mu1>
+      <mu2>0.7</mu2>
+      <kp>500000.0</kp>
+      <kd>10.0</kd>
+      <minDepth>0.002</minDepth>
+      <maxVel>0.1</maxVel>
+      <fdir1>1 0 0</fdir1>
+      <!-- <material>Gazebo/FlatBlack</material> -->
       <maxContacts>20</maxContacts>
     </gazebo>
@@ -43,5 +54,5 @@
       <origin xyz="${origin_x} ${origin_y} ${origin_z}" rpy="0 0 0" />
       <axis xyz="0 1 0" rpy="0 0 0" />
-      <limit effort="30" velocity="1.5"/>
+      <limit effort="-1" velocity="-1"/>
       <!-- <dynamics friction="0.5" damping="0.7" /> -->
     </joint>
