Commit message: wip: gazebo9 migration

File: hamster_vehicle_description/urdf/hamster.urdf.xacro (robot description, xacro)
@@ -1,467 +1,131 @@
 <?xml version="1.0"?>
 <robot name="agent" xmlns:xacro="http://www.ros.org/wiki/xacro">
-  <xacro:property name="degrees_45" value="0.785398163"/>
-  <xacro:property name="degrees_90" value="1.57079633"/>
-  <!-- chassis_length is measured along the x axis, chassis_width
-       along the y axis, and chassis_height along the z axis. -->
-  <xacro:property name="chassis_length" value="0.20"/>
-  <xacro:property name="chassis_width" value="0.06"/>
-  <xacro:property name="chassis_height" value="0.01"/>
-  <xacro:property name="chassis_mass" value="0.250"/>
-  <!-- hub_dia and tire_dia are the diameters of the hub and tire,
-       respectively. hex_hub_depth is the distance that the hex hub is
-       inset from the outer edge of the tire. It is set so that each wheel
-       is a "zero offset" wheel. hex_hub_depth = tire_width / 2 -
-       axle_length. -->
-  <xacro:property name="hub_dia" value="0.05"/>
-  <xacro:property name="tire_dia" value="0.20605"/>
-  <xacro:property name="tire_width" value="0.0889"/>
-  <xacro:property name="hex_hub_depth" value="0.01445"/>
-  <xacro:property name="wheel_mass" value="0.1"/>
-  <!-- hex_hub_dist is the distance between left and right hex hubs when
-       the shock absorbers are fully extended. axle_length is the distance
-       from a U joint to the corresponding hex hub. wheel_travel is the
-       vertical wheel travel. -->
-  <xacro:property name="wheelbase" value="0.165"/>
-  <xacro:property name="hex_hub_dist" value="0.20"/>
-  <xacro:property name="axle_length" value="0.03"/>
-  <xacro:property name="wheel_travel" value="0.01"/>
-  <xacro:property name="shock_z_offset" value="0.03"/>
-  <xacro:property name="axle_eff_limit" value="0.22766"/>
-  <xacro:property name="axle_vel_limit" value="15.8696"/>
-  <!-- These constants are used to simulate a Traxxas 2056 servo operated at
-       6 V. servo_stall_torque is measured in N m. servo_no_load_speed is
-       measured in rad/s. -->
-  <xacro:property name="servo_stall_torque" value="0.5649"/>
-  <xacro:property name="servo_no_load_speed" value="4.553"/>
-  <!-- Null inertial element. This is needed to make the model work with
-       Gazebo. -->
-  <xacro:macro name="null_inertial">
+  <xacro:include filename="$(find hamster_vehicle_description)/urdf/wheel.urdf.xacro" />
+    <xacro:macro name="solid_cuboid_inertia" params="w h d m">
+    <inertia  ixx="${m*(h*h+d*d)/12}" ixy = "0" ixz = "0"
+              iyy="${m*(w*w+d*d)/12}" iyz = "0"
+              izz="${m*(w*w+h*h)/12}" />
+    </xacro:macro>
+  <link name="base_link">
     <inertial>
-      <mass value="0.001"/>
-      <inertia ixx="0.001" ixy="0" ixz="0" iyy="0.001" iyz="0" izz="0.001"/>
+        <origin xyz="0 0 0" rpy="0 0 0" />
+        <mass value="1.0" />
+        <solid_cuboid_inertia w="0.1" h="0.1" d="0.2" m="1.0"/>
     </inertial>
-  </xacro:macro>
-  <!-- Inertia of a solid cuboid. Width is measured along the x axis, depth
-       along the y axis, and height along the z axis. -->
-  <xacro:macro name="solid_cuboid_inertial"
-               params="width depth height mass *origin">
-    <inertial>
-      <xacro:insert_block name="origin"/>
-      <mass value="${mass}"/>
-      <inertia ixx="${mass * (depth * depth + height * height) / 12}"
-               ixy="0" ixz="0"
-               iyy="${mass * (width * width + height * height) / 12}"
-               iyz="0"
-               izz="${mass * (width * width + depth * depth) / 12}"/>
-    </inertial>
-  </xacro:macro>
-  <!-- Inertia of a thick-walled cylindrical tube with open ends. Height is
-       measured along the z axis, which is the tube's axis. inner_rad and
-       outer_rad are the tube's inner and outer radii, respectively. -->
-  <xacro:macro name="thick_walled_tube_inertial"
-               params="inner_rad outer_rad height mass">
-    <inertial>
-      <mass value="${mass}"/>
-      <inertia ixx="${(1 / 12) * mass * (3 * (inner_rad * inner_rad +
-                    outer_rad * outer_rad) + height * height)}"
-               ixy="0" ixz="0"
-               iyy="${(1 / 12) * mass * (3 * (inner_rad * inner_rad +
-                    outer_rad * outer_rad) + height * height)}"
-               iyz="0"
-               izz="${mass * (inner_rad * inner_rad +
-                    outer_rad * outer_rad) / 2}"/>
-    </inertial>
-  </xacro:macro>
-  <!-- Shock absorber -->
-  <xacro:macro name="shock"
-               params="lr_prefix fr_prefix lr_reflect fr_reflect child">
-    <joint name="${lr_prefix}_${fr_prefix}_shock" type="fixed">
-      <parent link="chassis"/>
-      <child link="${child}"/>
-      <origin xyz="${fr_reflect * wheelbase / 2}
-                   ${lr_reflect * ((hex_hub_dist / 2) - axle_length)}
-                   ${(wheel_travel / 2) - shock_z_offset}"/>
-      <axis xyz="0 0 -1"/>
-      <limit lower="0" upper="0"
-             effort="0" velocity="0"/>
+    <surface>
+        <friction>
+          <ode>
+            <mu>1.0</mu>
+            <mu2>1.0</mu2>
+          </ode>
+        </friction>
+    </surface>
+    <visual>
+        <origin xyz="0 0 0.01" rpy="0 0 0" />
+        <geometry>
+            <mesh filename="package://hamster_vehicle_description/meshes/shell.dae" />
+        </geometry>
+    </visual>
+    <collision>
+        <origin xyz="-0.010 0 0.05"/>
+        <geometry>
+            <box size="0.25 0.09 0.05" />
+        </geometry>
+    </collision>
+  </link>
+  <link name="imu_link">
+        <inertial>
+            <mass value="0.01" />
+            <solid_cuboid_inertia w="0.05" h="0.05" d="0.07" m="0.01"/>
+        </inertial>
+        <visual>
+            <geometry>
+                <box size="0.01 0.01 0.01" />
+            </geometry>
+        </visual>
+    </link>
+    <joint name="imu_link_joint" type="fixed">
+        <origin xyz="0 0 0" rpy="0 0 0" />
+        <parent link="base_link" />
+        <child  link="imu_link" />
     </joint>
-  </xacro:macro>
-  <!-- The "wheel" macro defines an axle carrier, axle, and wheel. -->
-  <xacro:macro name="wheel" params="lr_prefix fr_prefix lr_reflect">
-    <link name="${lr_prefix}_${fr_prefix}_axle_carrier">
-      <xacro:null_inertial/>
-    </link>
-    <!-- The left and right axles have the same axis so that identical
-         rotation values cause the wheels to rotate in the same direction. -->
-    <joint name="${lr_prefix}_${fr_prefix}_axle" type="continuous">
-      <parent link="${lr_prefix}_${fr_prefix}_axle_carrier"/>
-      <child link="${lr_prefix}_${fr_prefix}_wheel"/>
-      <origin rpy="${degrees_90} 0 0"/>
-      <axis xyz="0 0 -1"/>
-      <limit effort="${axle_eff_limit}" velocity="${axle_vel_limit}"/>
-    </joint>
-    <transmission name="${lr_prefix}_${fr_prefix}_axle_trans">
-      <type>transmission_interface/SimpleTransmission</type>
-      <joint name="${lr_prefix}_${fr_prefix}_axle">
-	<hardwareInterface>EffortJointInterface</hardwareInterface>
-      </joint>
-      <actuator name="${lr_prefix}_${fr_prefix}_axle_act">
-        <hardwareInterface>EffortJointInterface</hardwareInterface>
-        <mechanicalReduction>1</mechanicalReduction>
-      </actuator>
-    </transmission>
-    <link name="${lr_prefix}_${fr_prefix}_wheel">
-      <visual>
-        <origin xyz="0
-                     ${lr_reflect * (axle_length - (tire_width /
-                     2 - hex_hub_depth))}
-                     0"/>
-        <geometry>
-	  <mesh filename="package://hamster_vehicle_description/meshes/wheel.dae" />
-        </geometry>
-      </visual>
-      <collision>
-        <origin xyz="0
-                     ${lr_reflect * (axle_length - (tire_width /
-                     2 - hex_hub_depth))}
-                     0"/>
-        <geometry>
-          <cylinder radius="0.032" length="0.035" />
-        </geometry>
-      </collision>
-      <xacro:thick_walled_tube_inertial
-          inner_rad="${hub_dia / 2}" outer_rad="${tire_dia / 2}"
-          height="${tire_width}" mass="${wheel_mass}"/>
-    </link>
-  </xacro:macro>
-  <!-- Front wheel -->
-  <xacro:macro name="front_wheel"
-               params="lr_prefix fr_prefix lr_reflect fr_reflect">
-    <xacro:shock lr_prefix="${lr_prefix}" fr_prefix="${fr_prefix}"
-                 lr_reflect="${lr_reflect}" fr_reflect="${fr_reflect}"
-                 child="${lr_prefix}_steering_link"/>
-    <link name="${lr_prefix}_steering_link">
-      <xacro:null_inertial/>
-    </link>
-    <joint name="${lr_prefix}_steering_joint" type="revolute">
-      <parent link="${lr_prefix}_steering_link"/>
-      <child link="${lr_prefix}_${fr_prefix}_axle_carrier"/>
-      <axis xyz="0 0 1"/>
-      <limit lower="${-degrees_45}" upper="${degrees_45}"
-             effort="${servo_stall_torque}" velocity="${servo_no_load_speed}"/>
-    </joint>
-    <transmission name="${lr_prefix}_steering_trans">
-      <type>transmission_interface/SimpleTransmission</type>
-      <joint name="${lr_prefix}_steering_joint">
-	<hardwareInterface>EffortJointInterface</hardwareInterface>
-      </joint>
-      <actuator name="${lr_prefix}_steering_act">
-        <hardwareInterface>EffortJointInterface</hardwareInterface>
-        <mechanicalReduction>1</mechanicalReduction>
-      </actuator>
-    </transmission>
-    <xacro:wheel lr_prefix="${lr_prefix}" fr_prefix="${fr_prefix}"
-                 lr_reflect="${lr_reflect}"/>
-  </xacro:macro>
-  <!-- Rear wheel -->
-  <xacro:macro name="rear_wheel"
-               params="lr_prefix fr_prefix lr_reflect fr_reflect">
-    <xacro:shock lr_prefix="${lr_prefix}" fr_prefix="${fr_prefix}"
-                 lr_reflect="${lr_reflect}" fr_reflect="${fr_reflect}"
-                 child="${lr_prefix}_${fr_prefix}_axle_carrier"/>
-    <xacro:wheel lr_prefix="${lr_prefix}" fr_prefix="${fr_prefix}"
-                 lr_reflect="${lr_reflect}"/>
-  </xacro:macro>
-  <!-- base_link must have geometry so that its axes can be displayed in
-       rviz. -->
-  <link name="base_link">
+      <joint name="hokuyo_joint" type="fixed">
+    <axis xyz="0 1 0" />
+    <origin xyz="0 0 ${height3 - axel_offset/2}" rpy="0 0 0"/>
+    <parent link="link3"/>
+    <child link="hokuyo_link"/>
+  </joint>
+  <!-- Hokuyo Laser -->
+  <link name="lidar_link">
+    <collision>
+      <origin xyz="0 0 0" rpy="0 0 0"/>
+      <geometry>
+    <box size="0.05 0.05 0.05"/>
+      </geometry>
+    </collision>
     <visual>
+      <origin xyz="0 0 0" rpy="0 0 0"/>
       <geometry>
-        <box size="0.001 0.001 0.001"/>
+        <mesh filename="package://hamster_vehicle_description/meshes/rp_lidar_head.dae" />
       </geometry>
     </visual>
-  </link>
-  <gazebo reference="base_link">
-    <material>Gazebo/Black</material>
-  </gazebo>
-  <!-- Chassis -->
-  <link name="chassis">
-    <visual>
-      <origin xyz="0 0 ${-chassis_height / 2 - 0.01}"/>
-      <geometry>
-        <box size="${chassis_length} ${chassis_width} ${chassis_height}"/>
-      </geometry>
-      <material name="ChassisColor">
-        <color rgba="0.08 0.08 0.08 1"/>
-      </material>
-    </visual>
-    <collision>
-      <origin xyz="0 0 ${-chassis_height / 2}"/>
-      <geometry>
-        <box size="${chassis_length} ${chassis_width} ${chassis_height}"/>
-      </geometry>
-    </collision>
-    <xacro:solid_cuboid_inertial
-        width="${chassis_length}" depth="${chassis_width}"
-        height="${chassis_height}" mass="${chassis_mass}">
-      <origin xyz="0 0 ${-chassis_height / 2}"/>
-    </xacro:solid_cuboid_inertial>
-  </link>
-  <gazebo reference="chassis">
-    <material>Gazebo/FlatBlack</material>
-  </gazebo>
-  <joint name="base_link_to_chasis" type="fixed">
-    <parent link="base_link"/>
-    <child link="chassis"/>
-  </joint>
-  <!-- Body -->
-  <link name="body">
-    <visual name="visual">
-      <origin xyz="0 0 0.0" rpy="0 0.05 0"/>
-      <geometry>
-        <mesh filename="package://hamster_vehicle_description/meshes/shell.stl" />
-      </geometry>
-      <material name="ShellColor">
-        <color rgba="0.08 0.08 0.08 1"/>
-      </material>
-    </visual>
-    <collision name="collision">
-      <origin xyz="0 0 0.00"/>
-      <geometry>
-	<mesh filename="package://hamster_vehicle_description/meshes/shell.stl" />
-      </geometry>
-    </collision>
     <inertial>
-      <mass value="0.00001"/>
-      <inertia ixx="0.00001" ixy="0" ixz="0" iyy="0.00001" iyz="0" izz="0.00001"/>
+      <mass value="1e-5" />
+      <origin xyz="0 0 0" rpy="0 0 0"/>
+      <inertia ixx="1e-6" ixy="0" ixz="0" iyy="1e-6" iyz="0" izz="1e-6" />
     </inertial>
   </link>
-  <joint name="chasis_to_body" type="fixed">
-    <origin xyz="0.005 0 -0.027"/>
-    <parent link="chassis"/>
-    <child link="body"/>
-  </joint>
-  <gazebo reference="body">
-    <material>Gazebo/FlatBlack</material>
+  <wheel fr="front" lr="right" parent="base_link" origin_x="0.08" origin_y="-0.086" origin_z="0.03"/>
+  <wheel fr="front" lr="left" parent="base_link" origin_x="0.08" origin_y="0.086" origin_z="0.03"/>
+  <wheel fr="rear" lr="right" parent="base_link" origin_x="-0.085" origin_y="-0.086" origin_z="0.03"/>
+  <wheel fr="rear" lr="left" parent="base_link" origin_x="-0.085" origin_y="0.086" origin_z="0.03"/>
+  <gazebo>
+    <plugin name="gazebo_ros_control" filename="libgazebo_ros_control.so">
+        <robotNamespace>/</robotNamespace>
+        <robotSimType>gazebo_ros_control/DefaultRobotHWSim</robotSimType>
+        <legacyModeNS>true</legacyModeNS>
+    </plugin>
   </gazebo>
-  <link name="laser_hokuyo">
-    <visual>
-      <geometry>
-        <box size="0.001 0.001 0.001"/>
-      </geometry>
-    </visual>
-    <collision>
-      <geometry>
-        <box size="0.001 0.001 0.001"/>
-      </geometry>
-    </collision>
-  </link>
-  <joint name="body_to_laser_hokuyo" type="fixed">
-    <origin xyz="-0.045 0.0 0.103"/>
-    <parent link="body"/>
-    <child link="laser_hokuyo"/>
-  </joint>
-  <link name="tag">
-    <visual>
-      <geometry>
-        <mesh filename="package://hamster_vehicle_description/meshes/tag.stl" />
-      </geometry>
-      <material name="TagColor">
-        <color rgba="0.5 0.0 0.0 1"/>
-      </material>
-    </visual>
-  </link>
-  <joint name="tag_to_body" type="fixed">
-    <origin xyz="0.0 0.0 0.0"/>
-    <parent link="body"/>
-    <child link="tag"/>
-  </joint>
-  <gazebo reference="tag">
-    <material>Gazebo/Red</material>
+            <!-- Skid steer drive controller -->
+  <gazebo>
+      <plugin name="skid_steer_drive_controller" filename="libgazebo_ros_skid_steer_drive.so">
+          <alwaysOn>1</alwaysOn>
+          <updateRate>100.0</updateRate>
+          <robotNamespace>/</robotNamespace>
+          <leftFrontJoint>front_left_wheel_joint</leftFrontJoint>
+          <rightFrontJoint>front_right_wheel_joint</rightFrontJoint>
+          <leftRearJoint>rear_left_wheel_joint</leftRearJoint>
+          <rightRearJoint>rear_right_wheel_joint</rightRearJoint>
+          <wheelSeparation>0.18</wheelSeparation>
+          <wheelDiameter>0.058</wheelDiameter>
+          <torque>50</torque>
+          <broadcastTF>0</broadcastTF>
+          <odometryFrame>map</odometryFrame>
+          <commandTopic>cmd_vel</commandTopic>
+          <odometryTopic>odom</odometryTopic>
+          <robotBaseFrame>base_link</robotBaseFrame>
+          <covariance_x>0.0001</covariance_x>
+          <covariance_y>0.0001</covariance_y>
+          <covariance_z>0.0001</covariance_z>
+          <covariance_yaw>0.0001</covariance_yaw>
+      </plugin>
   </gazebo>
-  <link name="camera">
-    <visual>
-      <geometry>
-        <mesh filename="package://hamster_vehicle_description/meshes/camera.stl" />
-      </geometry>
-      <material name="CameraColor">
-        <color rgba="0.2 0.0 0.0 1"/>
-      </material>
-    </visual>
-  </link>
-  <joint name="body_to_camera" type="fixed">
-    <origin xyz="0.1 0.0 -0.01"/>
-    <parent link="chassis"/>
-    <child link="camera"/>
-  </joint>
-  <gazebo reference="camera">
-    <material>Gazebo/Red</material>
-  </gazebo>
-  <link name="iris">
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
Commit message: loading urdf in namespace fixed

File: hamster_vehicle_description/urdf/hamster.urdf.xacro (robot description, xacro)
@@ -7,4 +7,5 @@
               izz="${m*(w*w+h*h)/12}" />
     </xacro:macro>
+  <xacro:arg name="agent" default="agent1" />
   <link name="base_link">
     <inertial>
@@ -50,9 +51,9 @@
         <child  link="imu_link" />
     </joint>
-      <joint name="hokuyo_joint" type="fixed">
+  <joint name="hokuyo_joint" type="fixed">
     <axis xyz="0 1 0" />
-    <origin xyz="0 0 ${height3 - axel_offset/2}" rpy="0 0 0"/>
-    <parent link="link3"/>
-    <child link="hokuyo_link"/>
+    <origin xyz="-0.05 0 0.115" rpy="0 0 0"/>
+    <parent link="base_link"/>
+    <child link="lidar_link"/>
   </joint>
   <!-- Hokuyo Laser -->
@@ -82,5 +83,5 @@
   <gazebo>
     <plugin name="gazebo_ros_control" filename="libgazebo_ros_control.so">
-        <robotNamespace>/</robotNamespace>
+        <robotNamespace>$(arg agent)</robotNamespace>
         <robotSimType>gazebo_ros_control/DefaultRobotHWSim</robotSimType>
         <legacyModeNS>true</legacyModeNS>
@@ -92,5 +93,5 @@
           <alwaysOn>1</alwaysOn>
           <updateRate>100.0</updateRate>
-          <robotNamespace>/</robotNamespace>
+          <robotNamespace>$(arg agent)</robotNamespace>
           <leftFrontJoint>front_left_wheel_joint</leftFrontJoint>
           <rightFrontJoint>front_right_wheel_joint</rightFrontJoint>
