Commit message: wip: realsense camera added

File: hamster_vehicle_description/urdf/hamster.urdf.xacro (robot description, xacro)
@@ -2,63 +2,65 @@
 <robot name="agent" xmlns:xacro="http://www.ros.org/wiki/xacro">
   <xacro:include filename="$(find hamster_vehicle_description)/urdf/wheel.urdf.xacro" />
-    <xacro:macro name="solid_cuboid_inertia" params="w h d m">
-    <inertia  ixx="${m*(h*h+d*d)/12}" ixy = "0" ixz = "0"
-              iyy="${m*(w*w+d*d)/12}" iyz = "0"
-              izz="${m*(w*w+h*h)/12}" />
-    </xacro:macro>
+  <xacro:macro name="solid_cuboid_inertia" params="w h d m">
+  <inertia  ixx="${m*(h*h+d*d)/12}" ixy = "0" ixz = "0"
+            iyy="${m*(w*w+d*d)/12}" iyz = "0"
+            izz="${m*(w*w+h*h)/12}" />
+  </xacro:macro>
   <xacro:arg name="agent" default="agent1" />
   <link name="base_link">
     <inertial>
-        <origin xyz="0 0 0" rpy="0 0 0" />
-        <mass value="1.0" />
-        <solid_cuboid_inertia w="0.1" h="0.1" d="0.2" m="1.0"/>
+      <mass value="1.0" />
+      <solid_cuboid_inertia w="0.1" h="0.1" d="0.2" m="1.0"/>
     </inertial>
     <surface>
-        <friction>
-          <ode>
-            <mu>1.0</mu>
-            <mu2>1.0</mu2>
-          </ode>
-        </friction>
+      <friction>
+        <ode>
+          <mu>1.0</mu>
+          <mu2>1.0</mu2>
+        </ode>
+      </friction>
     </surface>
     <visual>
-        <origin xyz="0 0 0.01" rpy="0 0 0" />
-        <geometry>
-            <mesh filename="package://hamster_vehicle_description/meshes/shell.dae" />
-        </geometry>
+      <geometry>
+        <mesh filename="package://hamster_vehicle_description/meshes/shell.dae" />
+      </geometry>
     </visual>
     <collision>
-        <origin xyz="-0.010 0 0.05"/>
-        <geometry>
-            <box size="0.25 0.09 0.05" />
-        </geometry>
+      <geometry>
+        <box size="0.25 0.09 0.05" />
+      </geometry>
     </collision>
   </link>
   <link name="imu_link">
-        <inertial>
-            <mass value="0.01" />
-            <solid_cuboid_inertia w="0.05" h="0.05" d="0.07" m="0.01"/>
-        </inertial>
-        <visual>
-            <geometry>
-                <box size="0.01 0.01 0.01" />
-            </geometry>
-        </visual>
+    <inertial>
+      <mass value="0.01" />
+      <solid_cuboid_inertia w="0.05" h="0.05" d="0.07" m="0.01"/>
+    </inertial>
+    <visual>
+      <geometry>
+        <box size="0.01 0.01 0.01" />
+      </geometry>
+    </visual>
     </link>
-    <joint name="imu_link_joint" type="fixed">
-        <origin xyz="0 0 0" rpy="0 0 0" />
-        <parent link="base_link" />
-        <child  link="imu_link" />
-    </joint>
+  <joint name="imu_link_joint" type="fixed">
+    <origin xyz="0 0 0" rpy="0 0 0" />
+    <parent link="base_link" />
+    <child  link="imu_link" />
+  </joint>
   <joint name="hokuyo_joint" type="fixed">
     <axis xyz="0 1 0" />
-    <origin xyz="-0.05 0 0.115" rpy="0 0 0"/>
+    <origin xyz="-0.05 0 0.085" rpy="0 0 0"/>
     <parent link="base_link"/>
     <child link="lidar_link"/>
+  </joint>
+  <joint name="camera_joint" type="fixed">
+    <axis xyz="0 1 0" />
+    <origin xyz="0.12673 0 0.028" rpy="1.57 0 1.57"/>
+    <parent link="base_link"/>
+    <child link="camera_link"/>
   </joint>
   <!-- Hokuyo Laser -->
   <link name="lidar_link">
     <collision>
-      <origin xyz="0 0 0" rpy="0 0 0"/>
       <geometry>
     <box size="0.05 0.05 0.05"/>
@@ -66,5 +68,4 @@
     </collision>
     <visual>
-      <origin xyz="0 0 0" rpy="0 0 0"/>
       <geometry>
         <mesh filename="package://hamster_vehicle_description/meshes/rp_lidar_head.dae" />
@@ -73,42 +74,58 @@
     <inertial>
       <mass value="1e-5" />
-      <origin xyz="0 0 0" rpy="0 0 0"/>
       <inertia ixx="1e-6" ixy="0" ixz="0" iyy="1e-6" iyz="0" izz="1e-6" />
     </inertial>
   </link>
-  <wheel fr="front" lr="right" parent="base_link" origin_x="0.08" origin_y="-0.086" origin_z="0.03"/>
-  <wheel fr="front" lr="left" parent="base_link" origin_x="0.08" origin_y="0.086" origin_z="0.03"/>
-  <wheel fr="rear" lr="right" parent="base_link" origin_x="-0.085" origin_y="-0.086" origin_z="0.03"/>
-  <wheel fr="rear" lr="left" parent="base_link" origin_x="-0.085" origin_y="0.086" origin_z="0.03"/>
+    <link name="camera_link">
+    <collision>
+      <geometry>
+    <box size="0.01 0.01 0.01"/>
+      </geometry>
+    </collision>
+    <visual>
+      <geometry>
+        <mesh filename="package://hamster_vehicle_description/meshes/d415.stl" />
+      </geometry>
+      <material name="red"/>
+    </visual>
+    <inertial>
+      <mass value="1e-5" />
+      <inertia ixx="1e-6" ixy="0" ixz="0" iyy="1e-6" iyz="0" izz="1e-6" />
+    </inertial>
+  </link>
+  <wheel fr="front" lr="right" parent="base_link" origin_x="0.08" origin_y="-0.086" origin_z="-0.01"/>
+  <wheel fr="front" lr="left" parent="base_link" origin_x="0.08" origin_y="0.086" origin_z="-0.01"/>
+  <wheel fr="rear" lr="right" parent="base_link" origin_x="-0.085" origin_y="-0.086" origin_z="-0.01"/>
+  <wheel fr="rear" lr="left" parent="base_link" origin_x="-0.085" origin_y="0.086" origin_z="-0.01"/>
   <gazebo>
     <plugin name="gazebo_ros_control" filename="libgazebo_ros_control.so">
-        <robotNamespace>$(arg agent)</robotNamespace>
-        <robotSimType>gazebo_ros_control/DefaultRobotHWSim</robotSimType>
-        <legacyModeNS>true</legacyModeNS>
+      <robotNamespace>$(arg agent)</robotNamespace>
+      <robotSimType>gazebo_ros_control/DefaultRobotHWSim</robotSimType>
+      <legacyModeNS>true</legacyModeNS>
     </plugin>
   </gazebo>
             <!-- Skid steer drive controller -->
   <gazebo>
-      <plugin name="skid_steer_drive_controller" filename="libgazebo_ros_skid_steer_drive.so">
-          <alwaysOn>1</alwaysOn>
-          <updateRate>100.0</updateRate>
-          <robotNamespace>$(arg agent)</robotNamespace>
-          <leftFrontJoint>front_left_wheel_joint</leftFrontJoint>
-          <rightFrontJoint>front_right_wheel_joint</rightFrontJoint>
-          <leftRearJoint>rear_left_wheel_joint</leftRearJoint>
-          <rightRearJoint>rear_right_wheel_joint</rightRearJoint>
-          <wheelSeparation>0.18</wheelSeparation>
-          <wheelDiameter>0.058</wheelDiameter>
-          <torque>50</torque>
-          <broadcastTF>0</broadcastTF>
-          <odometryFrame>map</odometryFrame>
-          <commandTopic>cmd_vel</commandTopic>
-          <odometryTopic>odom</odometryTopic>
-          <robotBaseFrame>base_link</robotBaseFrame>
-          <covariance_x>0.0001</covariance_x>
-          <covariance_y>0.0001</covariance_y>
-          <covariance_z>0.0001</covariance_z>
-          <covariance_yaw>0.0001</covariance_yaw>
-      </plugin>
+    <plugin name="skid_steer_drive_controller" filename="libgazebo_ros_skid_steer_drive.so">
+      <alwaysOn>1</alwaysOn>
+      <updateRate>100.0</updateRate>
+      <robotNamespace>$(arg agent)</robotNamespace>
+      <leftFrontJoint>front_left_wheel_joint</leftFrontJoint>
+      <rightFrontJoint>front_right_wheel_joint</rightFrontJoint>
+      <leftRearJoint>rear_left_wheel_joint</leftRearJoint>
+      <rightRearJoint>rear_right_wheel_joint</rightRearJoint>
+      <wheelSeparation>0.18</wheelSeparation>
+      <wheelDiameter>0.058</wheelDiameter>
+      <torque>50</torque>
+      <broadcastTF>0</broadcastTF>
+      <odometryFrame>map</odometryFrame>
+      <commandTopic>cmd_vel</commandTopic>
+      <odometryTopic>odom</odometryTopic>
+      <robotBaseFrame>base_link</robotBaseFrame>
+      <covariance_x>0.0001</covariance_x>
+      <covariance_y>0.0001</covariance_y>
+      <covariance_z>0.0001</covariance_z>
+      <covariance_yaw>0.0001</covariance_yaw>
+    </plugin>
   </gazebo>
   <gazebo reference="imu_link">
@@ -120,5 +137,5 @@
       <topic>__default_topic__</topic>
       <plugin filename="libgazebo_ros_imu_sensor.so" name="imu_plugin">
-        <topicName>sensors/imu_raw</topicName>
+        <topicName>$(arg agent)/imu</topicName>
         <bodyName>imu_link</bodyName>
         <updateRateHZ>10.0</updateRateHZ>
@@ -126,7 +143,79 @@
         <xyzOffset>0 0 0</xyzOffset>
         <rpyOffset>0 0 0</rpyOffset>
-        <frameName>imu_link</frameName>
+        <frameName>$(arg agent)/imu_link</frameName>
       </plugin>
     </sensor>
   </gazebo>
+  <gazebo reference="lidar_link">
+    <sensor type="gpu_ray" name="head_hokuyo_sensor">
+      <pose>0 0 0 0 0 0</pose>
+      <visualize>false</visualize>
+      <update_rate>40</update_rate>
+      <ray>
+        <scan>
+          <horizontal>
+            <samples>720</samples>
+            <resolution>1</resolution>
+            <min_angle>-3.1415</min_angle>
+            <max_angle>3.1415</max_angle>
+          </horizontal>
+        </scan>
+        <range>
+          <min>0.10</min>
+          <max>30.0</max>
+          <resolution>0.01</resolution>
+        </range>
+        <noise>
+          <type>gaussian</type>
+          <mean>0.0</mean>
+          <stddev>0.01</stddev>
+        </noise>
+      </ray>
+      <plugin name="gazebo_ros_head_hokuyo_controller" filename="libgazebo_ros_gpu_laser.so">
+        <topicName>$(arg agent)/scan</topicName>
+        <frameName>$(arg agent)/lidar_link</frameName>
+      </plugin>
+    </sensor>
+  </gazebo>
+  <gazebo reference="camera_link">
+    <sensor name="depth_camera" type="depth">
+      <update_rate>15</update_rate>
+      <camera>
+        <horizontal_fov>1.5882496</horizontal_fov>
+        <image>
+          <width>640</width>
+          <height>480</height>
+          <format>R8G8B8</format>
+        </image>
+        <clip>
+          <near>0.05</near>
+          <far>3</far>
+        </clip>
+      </camera>
+      <plugin name="camera_controller" filename="libgazebo_ros_openni_kinect.so">
+        <baseline>0.2</baseline>
+        <alwaysOn>true</alwaysOn>
+        <updateRate>1.0</updateRate>
+        <cameraName>$(arg agent)</cameraName>
+        <imageTopicName>camera/color/image_raw</imageTopicName>
+        <cameraInfoTopicName>camera/color/camera_info</cameraInfoTopicName>
+        <depthImageTopicName>camera/depth/image_raw</depthImageTopicName>
+        <depthImageInfoTopicName>camera/depth/camera_info</depthImageInfoTopicName>
+        <pointCloudTopicName>camera/depth/points</pointCloudTopicName>
+        <frameName>$(arg agent)/camera_link</frameName>
+        <pointCloudCutoff>0.5</pointCloudCutoff>
+        <pointCloudCutoffMax>3.0</pointCloudCutoffMax>
+        <distortionK1>0.00000001</distortionK1>
+        <distortionK2>0.00000001</distortionK2>
+        <distortionK3>0.00000001</distortionK3>
+        <distortionT1>0.00000001</distortionT1>
+        <distortionT2>0.00000001</distortionT2>
+        <CxPrime>0</CxPrime>
+        <Cx>0</Cx>
+        <Cy>0</Cy>
+        <focalLength>0</focalLength>
+        <hackBaseline>0</hackBaseline>
+      </plugin>
+    </sensor>
+  </gazebo>
 </robot>

Commit message: wip:ackermann drive

File: hamster_vehicle_description/urdf/hamster.urdf.xacro (robot description, xacro)
@@ -1,4 +1,4 @@
 <?xml version="1.0"?>
-<robot name="agent" xmlns:xacro="http://www.ros.org/wiki/xacro">
+<robot name="hamster" xmlns:xacro="http://www.ros.org/wiki/xacro">
   <xacro:include filename="$(find hamster_vehicle_description)/urdf/wheel.urdf.xacro" />
   <xacro:macro name="solid_cuboid_inertia" params="w h d m">
@@ -98,4 +98,14 @@
   <wheel fr="rear" lr="right" parent="base_link" origin_x="-0.085" origin_y="-0.086" origin_z="-0.01"/>
   <wheel fr="rear" lr="left" parent="base_link" origin_x="-0.085" origin_y="0.086" origin_z="-0.01"/>
+  <joint name="front_right_wheel_steering_joint" type="continuous">
+    <parent link="${parent}"/>
+    <child link="front_right_wheel_steering"/>
+    <axis xyz="0 0 0" rpy="0 0 0" />
+  </joint>
+  <joint name="front_left_wheel_steering_joint" type="continuous">
+    <parent link="${parent}"/>
+    <child link="front_left_wheel_steering"/>
+    <axis xyz="0 0 0" rpy="0 0 0" />
+  </joint>
   <gazebo>
     <plugin name="gazebo_ros_control" filename="libgazebo_ros_control.so">
@@ -107,5 +117,5 @@
             <!-- Skid steer drive controller -->
   <gazebo>
-    <plugin name="skid_steer_drive_controller" filename="libgazebo_ros_skid_steer_drive.so">
+    <!-- <plugin name="skid_steer_drive_controller" filename="libgazebo_ros_skid_steer_drive.so">
       <alwaysOn>1</alwaysOn>
       <updateRate>100.0</updateRate>
@@ -127,5 +137,5 @@
       <covariance_z>0.0001</covariance_z>
       <covariance_yaw>0.0001</covariance_yaw>
-    </plugin>
+    </plugin> -->
   </gazebo>
   <gazebo reference="imu_link">

Commit message: parameters server added

File: hamster_vehicle_description/urdf/hamster.urdf.xacro (robot description, xacro)
@@ -75,5 +75,5 @@
     <visual>
       <geometry>
-        <mesh filename="package://hamster_vehicle_description/meshes/rp_lidar_head.dae" />
+        <mesh filename="package://hamster_vehicle_description/meshes/rp_lidar_head.stl" />
       </geometry>
     </visual>
@@ -120,4 +120,16 @@
     <plugin name="gazebo_ackermann_drive" filename="libgazebo_ackermann_drive.so" >
       <robotNamespace>$(arg agent)</robotNamespace>
+      <wheelRadius>0.029</wheelRadius>
+      <frontLeftWheelJoint>front_left_wheel_joint</frontLeftWheelJoint>
+      <frontRightWheelJoint>front_right_wheel_joint</frontRightWheelJoint>
+      <reartLeftWheelJoint>rear_left_wheel_joint</reartLeftWheelJoint>
+      <rearRightWheelJoint>rear_right_wheel_joint</rearRightWheelJoint>
+      <frontRightWheelSteeringJoint>front_right_wheel_steering_joint</frontRightWheelSteeringJoint>
+      <frontLeftWheelSteeringJoint>front_left_wheel_steering_joint</frontLeftWheelSteeringJoint>
+      <torque>0.01</torque>
+      <baseFrame>$(arg agent)/base_link</baseFrame>
+      <odomFrame>$(arg agent)/odom/<odomFrame>
+      <odomTopic>odom</odomTopic>
+      <driveTopic>ackermann_cmd</driveTopic>
     </plugin>
   </gazebo>

Commit message: lidar improved, base link bug fixed

File: hamster_vehicle_description/urdf/hamster.urdf.xacro (robot description, xacro)
@@ -51,5 +51,5 @@
   <joint name="hokuyo_joint" type="fixed">
     <axis xyz="0 1 0" />
-    <origin xyz="-0.05 0 0.085" rpy="0 0 0"/>
+    <origin xyz="-0.05 0 0.06" rpy="0 0 0"/>
     <parent link="base_link"/>
     <child link="lidar_link"/>
@@ -75,5 +75,5 @@
     <visual>
       <geometry>
-        <mesh filename="package://hamster_vehicle_description/meshes/rp_lidar_head.stl" />
+        <mesh filename="package://hamster_vehicle_description/meshes/A2_lidar.dae" />
       </geometry>
     </visual>
@@ -118,7 +118,10 @@
             <!-- Skid steer drive controller -->
   <gazebo>
-    <plugin name="gazebo_ackermann_drive" filename="libgazebo_ackermann_drive.so" >
+    <plugin name="gazebo_ackermann_drive" filename="libgazebo_ackermann_drive.so">
       <robotNamespace>$(arg agent)</robotNamespace>
+      <robotBaseLink>base_link</robotBaseLink>
       <wheelRadius>0.029</wheelRadius>
+      <lateralSeparation>0.17</lateralSeparation>
+      <longitudalSeparation>0.166</longitudalSeparation>
       <frontLeftWheelJoint>front_left_wheel_joint</frontLeftWheelJoint>
       <frontRightWheelJoint>front_right_wheel_joint</frontRightWheelJoint>
@@ -128,6 +131,6 @@
       <frontLeftWheelSteeringJoint>front_left_wheel_steering_joint</frontLeftWheelSteeringJoint>
       <torque>0.01</torque>
-      <baseFrame>$(arg agent)/base_link</baseFrame>
-      <odomFrame>$(arg agent)/odom/<odomFrame>
+      <baseFrame>base_link</baseFrame>
+      <odomFrame>odom</odomFrame>
       <odomTopic>odom</odomTopic>
       <driveTopic>ackermann_cmd</driveTopic>
@@ -182,4 +185,5 @@
       </plugin>
     </sensor>
+    <material>Gazebo/DarkGrey</material>
   </gazebo>
   <xacro:if value="${version == 'V7'}">

Commit message: lidar sensor origin changed

File: hamster_vehicle_description/urdf/hamster.urdf.xacro (robot description, xacro)
@@ -51,5 +51,5 @@
   <joint name="hokuyo_joint" type="fixed">
     <axis xyz="0 1 0" />
-    <origin xyz="-0.05 0 0.06" rpy="0 0 0"/>
+    <origin xyz="-0.05 0 0.09" rpy="0 0 0"/>
     <parent link="base_link"/>
     <child link="lidar_link"/>
@@ -68,9 +68,4 @@
   <!-- Hokuyo Laser -->
   <link name="lidar_link">
-    <collision>
-      <geometry>
-    <box size="0.05 0.05 0.05"/>
-      </geometry>
-    </collision>
     <visual>
       <geometry>
@@ -78,8 +73,4 @@
       </geometry>
     </visual>
-    <inertial>
-      <mass value="1e-5" />
-      <inertia ixx="1e-6" ixy="0" ixz="0" iyy="1e-6" iyz="0" izz="1e-6" />
-    </inertial>
   </link>
   <link name="camera_link">
@@ -129,5 +120,5 @@
       <frontRightWheelSteeringJoint>front_right_wheel_steering_joint</frontRightWheelSteeringJoint>
       <frontLeftWheelSteeringJoint>front_left_wheel_steering_joint</frontLeftWheelSteeringJoint>
-      <torque>0.02</torque>
+      <torque>0.01</torque>
       <baseFrame>base_link</baseFrame>
       <odomFrame>odom</odomFrame>
@@ -162,6 +153,6 @@
     <sensor type="gpu_ray" name="head_hokuyo_sensor">
       <pose>0 0 0 0 0 0</pose>
-      <visualize>false</visualize>
-      <update_rate>40</update_rate>
+      <visualize>true</visualize>
+      <update_rate>10</update_rate>
       <ray>
         <scan>

Commit message: wandering added

File: hamster_vehicle_description/urdf/hamster.urdf.xacro (robot description, xacro)
@@ -56,7 +56,6 @@
   </joint>
   <joint name="camera_joint" type="fixed">
-    <axis xyz="0 1 0" />
     <xacro:if value="${version == 'V7'}">
-      <origin xyz="0.12673 0 0.028" rpy="1.57 0 1.57"/>
+      <origin xyz="0.12673 0 0.028" rpy="0 0 0"/>
     </xacro:if>
       <xacro:if value="${version == 'V6'}">
@@ -66,4 +65,12 @@
     <child link="camera_link"/>
   </joint>
+  <xacro:if value="${version == 'V7'}">
+    <link name="camera_optical_frame_link"/>
+      <joint name="camera_optical_joint" type="fixed">
+        <origin xyz="0 0 0" rpy="-1.57 0 -1.57"/>
+        <parent link="camera_link"/>
+        <child link="camera_optical_frame_link"/>
+      </joint>
+  </xacro:if>
   <!-- Hokuyo Laser -->
   <link name="lidar_link">
@@ -127,5 +134,5 @@
       <odomNoiseMean>0.0</odomNoiseMean>
       <odomNoiseStddev>0.01</odomNoiseStddev>
-      <minSpeed>-1.2</minSpeed>
+      <minSpeed>0.1</minSpeed>
       <maxSpeed>1.2</maxSpeed>
       <hamsterRotationPattern>true</hamsterRotationPattern>
@@ -153,5 +160,5 @@
     <sensor type="gpu_ray" name="head_hokuyo_sensor">
       <pose>0 0 0 0 0 0</pose>
-      <visualize>true</visualize>
+      <visualize>false</visualize>
       <update_rate>10</update_rate>
       <ray>
@@ -191,9 +198,9 @@
             <width>640</width>
             <height>480</height>
-            <format>R8G8B8</format>
+            <format>B8G8R8</format>
           </image>
           <clip>
             <near>0.05</near>
-            <far>3</far>
+            <far>200</far>
           </clip>
         </camera>
@@ -201,5 +208,5 @@
           <baseline>0.2</baseline>
           <alwaysOn>true</alwaysOn>
-          <updateRate>1.0</updateRate>
+          <updateRate>30.0</updateRate>
           <cameraName></cameraName>
           <imageTopicName>camera/color/image_raw</imageTopicName>
@@ -208,7 +215,7 @@
           <depthImageInfoTopicName>camera/depth/camera_info</depthImageInfoTopicName>
           <pointCloudTopicName>camera/depth/points</pointCloudTopicName>
-          <frameName>$(arg agent)/camera_link</frameName>
+          <frameName>camera_optical_frame_link</frameName>
           <pointCloudCutoff>0.5</pointCloudCutoff>
-          <pointCloudCutoffMax>3.0</pointCloudCutoffMax>
+          <pointCloudCutoffMax>5.0</pointCloudCutoffMax>
           <distortionK1>0.00000001</distortionK1>
           <distortionK2>0.00000001</distortionK2>
